File: ModbusPlug_Circuit/CP2102N_USBtoUART.kicad_sch (KiCad schematic)
At the start: 0 parts

Commit message: Updated USB/PD and TTL circuit
Parts:
- added C3: 4.7uF|16V, Capacitor_SMD:C_0402_1005Metric, symbol Device:C
- added C4: 100nF|16V, Capacitor_SMD:C_0402_1005Metric, symbol Device:C
- added D1, D2, D3: RED LED, LED_SMD:LED_0402_1005Metric, symbol Device:LED
- added R2: 1k 5%, Resistor_SMD:R_0402_1005Metric, symbol Device:R
- added R3: 22.1k 5%, Resistor_SMD:R_0402_1005Metric, symbol Device:R
- added R4: 47k 5%, Resistor_SMD:R_0402_1005Metric, symbol Device:R
- added RN1: 1k 5%, Resistor_SMD:R_Array_Convex_4x0402, symbol Device:R_Network04_Split
- added U2: CP2102N-Axx-xQFN20, Package_DFN_QFN:SiliconLabs_QFN-20-1EP_3x3mm_P0.5mm_EP1.8x1.8mm, symbol Interface_USB:CP2102N-Axx-xQFN20
Connections:
- new net: D2.2 (A), RN1.1 (R1)
- new net: R3.2, R4.1, U2.8 (VBUS)
- new net: D3.2 (A), RN1.1 (R1)
- new net: D1.2 (A), RN1.1 (R1)
- new net: R2.2, U2.9 (~{RST})
- new net Din_+: U2.5 (D-)
- new net Din_-: U2.4 (D+)
- new net GND: C3.2, C4.2, D1.1 (K), R4.2, U2.12 (GND), U2.21 (GND), U2.3 (GND)
- new net RS485_DE: U2.1 (RS485/GPIO.1)
- new net RXT: D3.1 (K), U2.19 (~{RXT}/GPIO.3)
- new net TXT: D2.1 (K), U2.20 (~{TXT}/GPIO.2)
- new net UART_RX: U2.17 (RXD)
- new net UART_TX: U2.18 (TXD)
- new net VBUS_in: R3.1
- new net Vin: C3.1, C4.1, R2.1, RN1.2 (R1.2), RN1.3 (R2.2), RN1.4 (R3.2), U2.6 (VDD), U2.7 (VREGIN)
- no-connect marks 0 -> 8

Commit message: pushing V0.1
Parts:
- removed RN1: 1k 5%, Resistor_SMD:R_Array_Convex_4x0402, symbol Device:R_Network04_Split
- added RN2: R_Pack04, Resistor_SMD:R_Array_Convex_4x0402, symbol Device:R_Pack04
Connections:
- net Vin: now also RN2.2 (R2.1), RN2.3 (R3.1), RN2.4 (R4.1)
- net at D2.2 (A): now also RN2.5 (R4.2)
- net at D3.2 (A): now also RN2.6 (R3.2)
- net at D1.2 (A): now also RN2.7 (R2.2)
Other:
- note added: "YC122-JR-0710KL"

Commit message: pushing V0.1.1
Connections:
- net Vin renamed 3.3V_in
Changed lines of the file:
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@@
+	(wire
+		(pts
+			(xy 198.12 78.74) (xy 209.55 78.74)
+		)
+		(stroke
+			(width 0)
+			(type default)
+		)
+	)
 	(wire
 		(pts
@@
 		(pts
 			(xy 60.96 50.8) (xy 69.85 50.8)
-		)
-		(stroke
-			(width 0)
-			(type default)
-		)
-	)
-	(wire
-		(pts
-			(xy 198.12 66.04) (xy 198.12 78.74)
 		)
 		(stroke
@@
 		)
 	)
-	(label "Vin"
-		(at 198.12 66.04 0)
-		(effects
-			(font
-				(size 1.27 1.27)
-			)
-			(justify left bottom)
+	(label "3.3V_in"
+		(at 209.55 78.74 180)
+		(effects
+			(font
+				(size 1.27 1.27)
+			)
+			(justify right bottom)
 		)
 	)
@@
 		)
 	)
-	(hierarchical_label "Vin"
-		(shape input)
-		(at 60.96 50.8 180)
-		(effects
-			(font
-				(size 1.27 1.27)
-			)
-			(justify right)
-		)
-	)
 	(hierarchical_label "UART_RX"
 		(shape input)
@@
 		)
 	)
+	(hierarchical_label "3.3V_in"
+		(shape input)
+		(at 60.96 50.8 180)
+		(effects
+			(font
+				(size 1.27 1.27)
+			)
+			(justify right)
+		)
+	)

Commit message: pushing V0.1.3
Connections:
- net 3.3V_in: now also RN2.5 (R4.2), RN2.6 (R3.2), RN2.7 (R2.2); no longer RN2.2 (R2.1), RN2.3 (R3.1), RN2.4 (R4.1)
- net at D2.2 (A): now also RN2.4 (R4.1); no longer RN2.5 (R4.2)
- net at D3.2 (A): now also RN2.3 (R3.1); no longer RN2.6 (R3.2)
- net at D1.2 (A): now also RN2.2 (R2.1); no longer RN2.7 (R2.2)
Other:
- moved on the sheet: RN2
Changed lines of the file:
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@@
 	(symbol
 		(lib_id "Device:R_Pack04")
-		(at 189.23 81.28 90)
+		(at 189.23 81.28 270)
+		(mirror x)
 		(unit 1)
 		(exclude_from_sim no)
@@
 		(on_board yes)
 		(dnp no)
-		(fields_autoplaced yes)
 		(property "Reference" "RN2"
 			(at 189.23 72.39 90)

Commit message: pushing V0.1.4
Other:
- note added: "Part number : YC122-JR-0710KL"
- note removed: "YC122-JR-0710KL"
- title: (none) -> ModbusPlug
- moved on the sheet: C3, C4, D1, D2, D3, R2, R3, R4, RN2, U2
