File: ModbusPlug_Circuit/ModbusPlug_Circuit.kicad_pcb (KiCad board)
At the start: 2 copper layers, 11.2 x 25 mm, 21 parts, among them P1 USB_C_Plug, U1 MCP1700x-330xxTT, U2 CP2102N-Axx-xQFN20, U3 SN65HVD75DRBR

Commit message: pushing V0.1
Parts:
- removed RN1: 1k 5%, Resistor_SMD:R_Array_Convex_4x0402
- added R5: 22R, Resistor_SMD:R_0402_1005Metric, F.Cu at (139.8, 77.0)
- added R8: 22R, Resistor_SMD:R_0402_1005Metric, F.Cu at (157.6, 80.3)
- added RN2: R_Pack04, Resistor_SMD:R_Array_Convex_4x0402, B.Cu at (128.9, 75.0)
- added U4: USBLC6-2SC6, Package_TO_SOT_SMD:SOT-23-6, F.Cu at (126.1, 73.0)
- C1, C2, R1: moved to B.Cu
- R6, R7: value 5.1k 1% -> 10R 1%
- moved D3 24.2 mm to (131.1, 80.0)
- moved D2 24.0 mm to (131.1, 77.7)
- moved D1 23.9 mm to (131.1, 75.3)
- moved U3 11.3 mm to (140.0, 80.4)
- moved U2 7.21 mm to (126.6, 78.8)
- moved U1 5.66 mm to (130.8, 71.5)
- moved C2 3.83 mm to (127.8, 72.7), turned to 180 degrees
- moved C1 2.80 mm to (127.8, 71.5)
- moved R1 0.48 mm to (127.8, 70.5), turned to 180 degrees
Connections:
- C7 pad 1: unconnected-(C7-Pad1) -> /USB To UART/Vin
- C7 pad 2: unconnected-(C7-Pad2) -> GND
- P1 pad A6: /USB To UART/Din_+ -> /USB Type C & Power/D+
- P1 pad A7: /USB To UART/Din_- -> /USB Type C & Power/D-
- P1 pad B6: /USB To UART/Din_+ -> /USB Type C & Power/D+
- P1 pad B7: /USB To UART/Din_- -> /USB Type C & Power/D-
- U3 pad 1: unconnected-(U3-R-Pad1) -> Net-(U3-R)
- U3 pad 4: unconnected-(U3-D-Pad4) -> Net-(U3-D)
- U3 pad 5: unconnected-(U3-GND-Pad5) -> GND
- U3 pad 8: unconnected-(U3-VCC-Pad8) -> /USB To UART/Vin
- U3 pad 9: (no net) -> GND
Routing:
- net /USB Type C & Power/D+: track 0.00 -> 9.64 mm, vias 0 -> 2
- net /USB Type C & Power/D-: track 0.00 -> 7.71 mm
- net /USB To UART/Din_-: track 0.00 -> 3.56 mm
- net /USB To UART/Din_+: track 0.62 -> 3.56 mm

Commit message: pushing V0.1.1
Parts:
- added D4: SM712_SOT23, Package_TO_SOT_SMD:SOT-23, F.Cu at (131.0, 86.3)
- added R9: 120R 1%, Resistor_SMD:R_0402_1005Metric, F.Cu at (131.0, 81.6)
- added RN1: 10k 5%, Resistor_SMD:R_Array_Convex_2x0402, F.Cu at (143.0, 76.3)
- C5, C6: value 1uF|16V -> 330pF|50V
- R5, R8: value 22R -> 22R 1%
- moved R7 22.7 mm to (129.8, 81.1), turned to -90 degrees
- moved C5 20.2 mm to (129.8, 83.2), turned to -90 degrees
- moved R6 20.0 mm to (132.3, 81.1), turned to -90 degrees
- moved C6 17.2 mm to (132.4, 83.2), turned to -90 degrees
- moved U3 9.27 mm to (131.1, 77.9)
Connections:
- net /USB To UART/Vin renamed +3.3V
- net /USB Type C & Power/VBUS renamed /USB Type C & Power/VBUS_out
- C5 pad 1: unconnected-(C5-Pad1) -> /Modbus_Transciever/A+
- C5 pad 2: unconnected-(C5-Pad2) -> GND
- C6 pad 1: unconnected-(C6-Pad1) -> /Modbus_Transciever/B-
- C6 pad 2: unconnected-(C6-Pad2) -> GND
- R5 pad 1: unconnected-(R5-Pad1) -> /Modbus_Transciever/RS485_R
- R6 pad 1: unconnected-(R6-Pad1) -> Net-(U3-B)
- R6 pad 2: unconnected-(R6-Pad2) -> /Modbus_Transciever/B-
- R7 pad 1: unconnected-(R7-Pad1) -> Net-(U3-A)
- R7 pad 2: unconnected-(R7-Pad2) -> /Modbus_Transciever/A+
- R8 pad 1: unconnected-(R8-Pad1) -> /Modbus_Transciever/RS485_D
- U2 pad 1: /USB To UART/RS485_DE -> /Modbus_Transciever/RS485_DE
- U2 pad 17: /USB To UART/UART_RX -> /Modbus_Transciever/RS485_R
- U2 pad 18: /USB To UART/UART_TX -> /Modbus_Transciever/RS485_D
- U3 pad 2: unconnected-(U3-~{RE}-Pad2) -> /Modbus_Transciever/RS485_DE
- U3 pad 3: unconnected-(U3-DE-Pad3) -> /Modbus_Transciever/RS485_DE
- U3 pad 6: unconnected-(U3-A-Pad6) -> Net-(U3-A)
- U3 pad 7: unconnected-(U3-B-Pad7) -> Net-(U3-B)
Other:
- copper layers 2 -> 4

Commit message: pushin V0.1.2
Parts:
- added J1: Conn_01x01_Pin, Connector_Wire:SolderWirePad_1x01_SMD_1x2mm, F.Cu at (123.3, 90.0)
- added J2: Conn_01x01_Pin, Connector_Wire:SolderWirePad_1x01_SMD_1x2mm, F.Cu at (128.5, 90.0)
- C3, C4, C7, R2, R3, R4: moved to B.Cu
- moved R8 33.3 mm to (124.6, 76.1), turned to -90 degrees
- moved C3 32.5 mm to (128.7, 83.3)
- moved C4 30.9 mm to (128.7, 82.3)
- moved R2 26.1 mm to (132.6, 84.7)
- moved R4 23.9 mm to (128.2, 79.8), turned to -90 degrees
- moved R3 23.9 mm to (128.2, 77.8), turned to -90 degrees
- moved C7 22.1 mm to (127.2, 81.3), turned to -90 degrees
- moved R5 13.3 mm to (126.6, 76.1), turned to -90 degrees
- moved RN2 9.01 mm to (137.2, 71.5)
- moved U2 6.82 mm to (130.7, 84.3)
- moved R6 6.36 mm to (126.1, 82.5)
- moved R9 5.91 mm to (125.6, 84.0)
- moved C5 5.83 mm to (124.0, 83.5), turned to 90 degrees
- moved U3 5.68 mm to (125.6, 79.3)
- moved D4 5.44 mm to (125.6, 86.5)
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Routing:
- net /USB Type C & Power/VBUS_out: track 0.00 -> 4.34 mm, vias 0 -> 3
- net Net-(U2-~{RST}): track 0.00 -> 1.57 mm, vias 0 -> 1
- net Net-(U2-VBUS): track 0.00 -> 1.15 mm, vias 0 -> 1
- net /Modbus_Transciever/RS485_DE: track 0.00 -> 1.15 mm, vias 0 -> 1
- net /USB To UART/TXT: track 0.00 -> 1.09 mm, vias 0 -> 1
- net /USB To UART/RXT: track 0.00 -> 0.93 mm, vias 0 -> 1
- net /Modbus_Transciever/RS485_R: track 0.00 -> 0.91 mm, vias 0 -> 1
- net /Modbus_Transciever/RS485_D: track 0.00 -> 0.87 mm, vias 0 -> 1
- net /USB Type C & Power/D+: track 9.64 -> 9.05 mm
- net /USB To UART/Din_-: track 3.56 -> 3.05 mm
- net /USB To UART/Din_+: track 3.56 -> 3.05 mm
- net GND: vias 0 -> 4
Other:
- board size 11.2 x 25 mm -> 12 x 25.1 mm
- board text added: "Stackup: JLC04101H-7628 (Standard), 4-layer, 1.02 mm ±10%"

Commit message: pushing V0.1.3
Parts:
- added J3: Conn_01x01_Pin, Connector_Wire:SolderWirePad_1x01_SMD_1x2mm, F.Cu at (133.5, 89.7)
- RN1: moved to B.Cu
- moved RN1 17.1 mm to (125.9, 77.2), turned to -90 degrees
- moved RN2 4.91 mm to (132.3, 71.2), turned to 90 degrees
- moved R2 3.92 mm to (128.7, 85.1)
- moved C1 1.50 mm to (125.0, 71.5)
- moved C2 1.50 mm to (125.0, 72.7)
- moved R1 1.50 mm to (125.0, 70.5)
- moved R5 1.22 mm to (126.6, 74.8)
- moved R8 1.22 mm to (124.6, 74.8)
- moved R4 0.80 mm to (128.2, 79.0), turned to 180 degrees
- moved C3 0.75 mm to (128.7, 84.0)
- moved C4 0.75 mm to (128.7, 83.0)
- moved C7 0.55 mm to (127.2, 80.8)
- moved J1 0.36 mm to (123.5, 89.7)
- moved J2 0.30 mm to (128.5, 89.7)
- turned R3 to 0 degrees
Connections:
- RN1 pad 1: GND -> /Modbus_Transciever/RS485_DE
- RN1 pad 4: /Modbus_Transciever/RS485_DE -> GND
- RN2 pad 2: +3.3V -> Net-(D1-A)
- RN2 pad 3: +3.3V -> Net-(D3-A)
- RN2 pad 4: +3.3V -> Net-(D2-A)
- RN2 pad 5: Net-(D2-A) -> +3.3V
- RN2 pad 6: Net-(D3-A) -> +3.3V
- RN2 pad 7: Net-(D1-A) -> +3.3V
Routing:
- net /Modbus_Transciever/RS485_D: track 0.87 -> 27.5 mm, vias 1 -> 2
- net /Modbus_Transciever/RS485_R: track 0.91 -> 23.2 mm, vias 1 -> 2
- net /Modbus_Transciever/RS485_DE: track 1.15 -> 17.7 mm, vias 1 -> 2
- net +3.3V: track 0.00 -> 10.2 mm, vias 0 -> 14
- net /Modbus_Transciever/B-: track 0.00 -> 8.27 mm
- net Net-(D3-A): track 0.00 -> 7.94 mm, vias 0 -> 1
- net /Modbus_Transciever/A+: track 0.00 -> 7.35 mm
- net /USB To UART/TXT: track 1.09 -> 8.24 mm, vias 1 -> 0
- net Net-(U2-VBUS): track 1.15 -> 7.58 mm
- net /USB To UART/RXT: track 0.93 -> 5.23 mm, vias 1 -> 0
- net /USB To UART/Din_-: track 3.05 -> 7.30 mm
- net /USB To UART/Din_+: track 3.05 -> 7.30 mm
- net Net-(D2-A): track 0.00 -> 3.75 mm, vias 0 -> 1
- net Net-(RN1B-R2.1): track 0.00 -> 3.70 mm, vias 0 -> 1
- net Net-(P1-CC): track 0.00 -> 3.43 mm, vias 0 -> 1
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- added copper zone on B.Cu, net +3.3V
- added copper zone on F.Cu, net +3.3V
- added copper zone on In2.Cu, net +3.3V
- added copper zone on F.Cu, net /Modbus_Transciever/A+
- added copper zone on F.Cu, net /Modbus_Transciever/B-
- added copper zone on B.Cu, net /USB Type C & Power/VBUS_out
- added copper zone on F.Cu, net /USB Type C & Power/VBUS_out
- added copper zone on In2.Cu, net /USB Type C & Power/VBUS_out
- added copper zone on B.Cu, net GND
- added copper zone on F.Cu, net GND
- added copper zone on In1.Cu, net GND
Other:
- outline, holes or cut-outs redrawn

Commit message: pushing V0.1.4
Parts:
- added G***: LOGO, LOGO, F.Cu at (64.3, 104.0)
- added G***: LOGO, LOGO, B.Cu at (63.8, 114.2)
- added G***: LOGO, LOGO, B.Cu at (62.7, 122.5)
- moved C7 77.7 mm to (57.1, 114.4), turned to 180 degrees
- moved C1 76.9 mm to (55.9, 105.2)
- moved C2 76.9 mm to (55.9, 106.3)
- moved C3 76.9 mm to (59.6, 117.7)
- moved C4 76.9 mm to (59.6, 116.7)
- moved D4 76.9 mm to (56.5, 120.2)
- moved J1 76.9 mm to (54.4, 123.3)
- moved J2 76.9 mm to (59.4, 123.3)
- moved J3 76.9 mm to (64.4, 123.3)
- moved P1 76.9 mm to (59.4, 101.2)
- moved R1 76.9 mm to (55.9, 104.1)
- moved R4 76.9 mm to (59.1, 112.6)
- moved R5 76.9 mm to (57.5, 108.5)
- moved R9 76.9 mm to (56.5, 117.7)
- moved U2 76.9 mm to (61.6, 118.0)
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Routing:
- net GND: vias 32 -> 31
Other:
- board text added: "0"
- board text added: "0 mm"
- board text added: "0.0000 mm / 0.0000 mm"
- board text added: "0.0152 mm"
- board text added: "0.02"
- board text added: "0.035 mm"
- board text added: "0.2000 mm"
- board text added: "0.2104 mm"
- board text added: "0.5 mm"
- board text added: "1"
- board text added: "1.0212 mm"
- board text added: "12.0000 mm x 25.1000 mm"
- board text added: "3.3"
- board text added: "4"
- board text added: "4.5"
- board text added: "A"
- board text added: "B"
- board text added: "B.Cu"
- board text added: "B.Mask"
- board text added: "B.Paste"
- board text added: "B.Silkscreen"
- board text added: "BOARD CHARACTERISTICS"
- board text added: "Black"
- board text added: "Board Thickness:"
- board text added: "Board overall dimensions:"
- board text added: "Bottom Silk Screen"
- board text added: "Bottom Solder Mask"
- board text added: "Bottom Solder Paste"
- board text added: "Castellated pads:"
- board text added: "Color"
- board text added: "Copper Finish:"
- board text added: "Copper Layer Count:"
- board text added: "Dielectric"
- board text added: "Edge card connectors:"
- board text added: "Epsilon R"
- board text added: "F.Cu"
- board text added: "F.Mask"
- board text added: "F.Paste"
- board text added: "F.Silkscreen"
- board text added: "FR4"
- board text added: "FR4 natural"
- board text added: "GND"
- board text added: "HAL SnPb"
- board text added: "Impedance Control:"
- board text added: "In1.Cu"
- board text added: "In2.Cu"
- board text added: "Layer Name"
- board text added: "Loss Tangent"
- board text added: "Material"
- board text added: "Min hole diameter:"
- board text added: "Min track/spacing:"
- board text added: "No"
- board text added: "Not specified"
- board text added: "Plated Board Edge:"
- board text added: "Thickness (mm)"
- board text added: "Top Silk Screen"
- board text added: "Top Solder Mask"
- board text added: "Top Solder Paste"
- board text added: "Type"
- board text added: "V0.1.4"
- board text added: "White"
- board text added: "copper"
- board text added: "core"
- board text added: "prepreg"
